File: PressureSensor/Pressure_sensor/Pressure_sensor.kicad_pcb (KiCad board)
At the start: 2 copper layers, 132 x 80.8 mm, 78 parts, among them J1 Power Input, J2 Conn_01x04_Pin, J3 Screw_Terminal_01x03, J4 Conn_02x03_Odd_Even, J5 Valve Terminal, J6 Conn_01x05_Pin, J7 USB_A, K1 SANYOU_SRD_Form_C, Q1 BC848, SW1 SW_SPST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

Commit message: Push
Parts:
- removed U4: EA_T123X-I2C, Display:Adafruit_SSD1306_No_Mounting_Holes
- added U5: DM-OLED096-636, DM-OLED096-636:MODULE_DM-OLED096-636, F.Cu at (190.2, 82.1)
- D8: footprint Diode_SMD:D_SOD-523 -> Diode_SMD:D_SOD-123
- R20, R21: value 10K -> 2K2
- moved U2 353.6 mm to (153.5, 85.4), turned to 90 degrees
- moved D9 342.2 mm to (139.7, 99.7), turned to 180 degrees
- moved L1 332.3 mm to (154.6, 113.6), turned to -90 degrees
- moved C7 331.1 mm to (139.7, 113.5), turned to -90 degrees
- moved BT1 331.1 mm to (195.3, 73.9), turned to 90 degrees
- moved R17 322.9 mm to (165.7, 100.2), turned to 90 degrees
- moved R18 320.8 mm to (167.3, 100.2), turned to -90 degrees
- moved R15 320.4 mm to (168.9, 100.2), turned to -90 degrees
- moved C8 313.0 mm to (161.5, 100.1), turned to 90 degrees
- moved C9 310.6 mm to (163.4, 100.1), turned to 90 degrees
- moved C12 306.6 mm to (181.8, 118.3), turned to 180 degrees
- moved BT2 305.7 mm to (172.6, 73.9), turned to 90 degrees
- moved C13 305.1 mm to (181.8, 116.5), turned to 180 degrees
- moved C11 300.1 mm to (168.6, 113.7), turned to 90 degrees
- moved C10 295.6 mm to (181.8, 114.7), turned to 180 degrees
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Connections:
- net Net-(J6-Pin_4) renamed DTR
Other:
- board size 132 x 80.8 mm -> 79 x 96.3 mm
